File: Schematics/Final_Project_Schematic/Final_Project_Schematic.sch (KiCad schematic (older format))
At the start: 9 parts

Commit message: schematic of MSP432 created
Parts:
- added MCU: MSP432P401R, symbol MSP432:MSP432P401R
Connections:
- net labels added: 1.65V, ADC_In, V_In, V_Out
- wire segments 17 -> 26
Other:
- moved on the sheet: C, MK, Op-Amp, R
Changed lines of the file:
@@
 L Amplifier_Operational:OP1177AR Op-Amp
 U 1 1 607D08F5
-P 5500 3300
-F 0 "Op-Amp" H 5600 3200 50  0000 L CNN
-F 1 "MCP6231-E/P" H 5500 3100 50  0000 L CNN
-F 2 "" H 5500 3000 50  0001 C CNN
-F 3 "" H 5500 3300 50  0001 C CNN
-	1    5500 3300
+P 5600 3300
+F 0 "Op-Amp" H 5700 3200 50  0000 L CNN
+F 1 "MCP6231-E/P" H 5600 3100 50  0000 L CNN
+F 2 "" H 5600 3000 50  0001 C CNN
+F 3 "" H 5600 3300 50  0001 C CNN
+	1    5600 3300
 	1    0    0    -1
 $EndComp
@@
 L power:GND #PWR?
 U 1 1 607D1EE4
-P 5400 3600
-F 0 "#PWR?" H 5400 3350 50  0001 C CNN
-F 1 "GND" H 5405 3427 50  0000 C CNN
-F 2 "" H 5400 3600 50  0001 C CNN
-F 3 "" H 5400 3600 50  0001 C CNN
-	1    5400 3600
-	1    0    0    -1
-$EndComp
-$Comp
-L power:+3.3V #PWR?
-U 1 1 607D2385
-P 5400 3000
-F 0 "#PWR?" H 5400 2850 50  0001 C CNN
-F 1 "+3.3V" H 5415 3173 50  0000 C CNN
-F 2 "" H 5400 3000 50  0001 C CNN
-F 3 "" H 5400 3000 50  0001 C CNN
-	1    5400 3000
+P 5500 3600
+F 0 "#PWR?" H 5500 3350 50  0001 C CNN
+F 1 "GND" H 5505 3427 50  0000 C CNN
+F 2 "" H 5500 3600 50  0001 C CNN
+F 3 "" H 5500 3600 50  0001 C CNN
+	1    5500 3600
 	1    0    0    -1
 $EndComp
@@
 L Device:R_US R
 U 1 1 607D5469
-P 5400 2700
-F 0 "R" V 5195 2700 50  0000 C CNN
-F 1 "1MΩ" V 5286 2700 50  0000 C CNN
-F 2 "" V 5440 2690 50  0001 C CNN
-F 3 "~" H 5400 2700 50  0001 C CNN
-	1    5400 2700
+P 5500 2700
+F 0 "R" V 5295 2700 50  0000 C CNN
+F 1 "1MΩ" V 5386 2700 50  0000 C CNN
+F 2 "" V 5540 2690 50  0001 C CNN
+F 3 "~" H 5500 2700 50  0001 C CNN
+	1    5500 2700
 	0    1    1    0
 $EndComp
@@
 L Device:C C
 U 1 1 607D6315
-P 4200 3400
-F 0 "C" V 3950 3400 50  0000 C CNN
-F 1 "1uF" V 4050 3400 50  0000 C CNN
-F 2 "" H 4238 3250 50  0001 C CNN
-F 3 "~" H 4200 3400 50  0001 C CNN
-	1    4200 3400
+P 4300 3400
+F 0 "C" V 4050 3400 50  0000 C CNN
+F 1 "1uF" V 4150 3400 50  0000 C CNN
+F 2 "" H 4338 3250 50  0001 C CNN
+F 3 "~" H 4300 3400 50  0001 C CNN
+	1    4300 3400
 	0    1    1    0
 $EndComp
@@
 L Device:R_US R
 U 1 1 607D2956
-P 3900 3250
-F 0 "R" H 3968 3296 50  0000 L CNN
-F 1 "2kΩ" H 3968 3205 50  0000 L CNN
-F 2 "" V 3940 3240 50  0001 C CNN
-F 3 "~" H 3900 3250 50  0001 C CNN
-	1    3900 3250
+P 4000 3250
+F 0 "R" H 4068 3296 50  0000 L CNN
+F 1 "2kΩ" H 4068 3205 50  0000 L CNN
+F 2 "" V 4040 3240 50  0001 C CNN
+F 3 "~" H 4000 3250 50  0001 C CNN
+	1    4000 3250
 	1    0    0    -1
 $EndComp
@@
 L Device:Microphone MK
 U 1 1 607D13BF
-P 3750 3600
-F 0 "MK" H 3500 3650 50  0000 L CNN
-F 1 "CMA-4544PF-W" H 3000 3500 50  0000 L CNN
-F 2 "" V 3750 3700 50  0001 C CNN
-F 3 "~" V 3750 3700 50  0001 C CNN
-	1    3750 3600
+P 3850 3600
+F 0 "MK" H 3600 3650 50  0000 L CNN
+F 1 "CMA-4544PF-W" H 3100 3500 50  0000 L CNN
+F 2 "" V 3850 3700 50  0001 C CNN
+F 3 "~" V 3850 3700 50  0001 C CNN
+	1    3850 3600
 	1    0    0    -1
 $EndComp
@@
 L Device:R_US R
 U 1 1 607EA2D2
-P 5400 2400
-F 0 "R" V 5195 2400 50  0000 C CNN
-F 1 "1MΩ" V 5286 2400 50  0000 C CNN
-F 2 "" V 5440 2390 50  0001 C CNN
-F 3 "~" H 5400 2400 50  0001 C CNN
-	1    5400 2400
-	0    1    1    0
-$EndComp
-Wire Wire Line
-	3750 3400 3900 3400
-Wire Wire Line
-	3900 3400 4050 3400
-Connection ~ 3900 3400
-Wire Wire Line
-	4350 3400 4450 3400
-Wire Wire Line
-	4750 3400 5100 3400
-Wire Wire Line
-	5200 3200 4900 3200
+P 5500 2400
+F 0 "R" V 5295 2400 50  0000 C CNN
+F 1 "1MΩ" V 5386 2400 50  0000 C CNN
+F 2 "" V 5540 2390 50  0001 C CNN
+F 3 "~" H 5500 2400 50  0001 C CNN
+	1    5500 2400
+	0    1    1    0
+$EndComp
+Wire Wire Line
+	3850 3400 4000 3400
+Wire Wire Line
+	4000 3400 4150 3400
+Connection ~ 4000 3400
+Wire Wire Line
+	4750 3400 5050 3400
 Wire Wire Line
 	4900 3100 4900 3200
 Wire Wire Line
-	5800 3300 5950 3300
-Wire Wire Line
-	5950 3300 5950 2550
-Wire Wire Line
-	5950 2550 5550 2550
-Wire Wire Line
-	5550 2550 5550 2700
-Wire Wire Line
-	5550 2400 5550 2550
-Connection ~ 5550 2550
-Wire Wire Line
-	5250 2700 5250 2550
-Wire Wire Line
-	5250 2550 5100 2550
-Wire Wire Line
-	5100 2550 5100 3400
-Connection ~ 5250 2550
-Wire Wire Line
-	5250 2550 5250 2400
-Connection ~ 5100 3400
-Wire Wire Line
-	5100 3400 5200 3400
-$Comp
-L power:+3.3V #PWR?
-U 1 1 607EC2B1
-P 4900 2800
-F 0 "#PWR?" H 4900 2650 50  0001 C CNN
-F 1 "+3.3V" H 4915 2973 50  0000 C CNN
-F 2 "" H 4900 2800 50  0001 C CNN
-F 3 "" H 4900 2800 50  0001 C CNN
-	1    4900 2800
-	1    0    0    -1
-$EndComp
-$Comp
-L power:+3.3V #PWR?
-U 1 1 607ECA78
-P 3900 3100
-F 0 "#PWR?" H 3900 2950 50  0001 C CNN
-F 1 "+3.3V" H 3915 3273 50  0000 C CNN
-F 2 "" H 3900 3100 50  0001 C CNN
-F 3 "" H 3900 3100 50  0001 C CNN
-	1    3900 3100
-	1    0    0    -1
-$EndComp
+	5900 3300 6150 3300
+Wire Wire Line
+	6150 3300 6150 2550
+Wire Wire Line
+	6150 2550 5650 2550
+Wire Wire Line
+	5650 2550 5650 2700
+Wire Wire Line
+	5650 2400 5650 2550
+Connection ~ 5650 2550
+Wire Wire Line
+	5350 2700 5350 2550
+Wire Wire Line
+	5350 2550 5050 2550
+Connection ~ 5350 2550
+Wire Wire Line
+	5350 2550 5350 2400
+Connection ~ 5050 3400
+Wire Wire Line
+	5050 3400 5300 3400
 $Comp
 L power:GND #PWR?
@@
 L power:GND #PWR?
 U 1 1 607ED134
-P 3750 3800
-F 0 "#PWR?" H 3750 3550 50  0001 C CNN
-F 1 "GND" H 3755 3627 50  0000 C CNN
-F 2 "" H 3750 3800 50  0001 C CNN
-F 3 "" H 3750 3800 50  0001 C CNN
-	1    3750 3800
+P 3850 3800
+F 0 "#PWR?" H 3850 3550 50  0001 C CNN
+F 1 "GND" H 3855 3627 50  0000 C CNN
+F 2 "" H 3850 3800 50  0001 C CNN
+F 3 "" H 3850 3800 50  0001 C CNN
+	1    3850 3800
 	1    0    0    -1
 $EndComp
@@
 Wire Wire Line
 	4900 3200 4900 3500
+$Comp
+L MSP432:MSP432P401R MCU
+U 1 1 60818468
+P 7150 3250
+F 0 "MCU" H 7150 1327 50  0000 C CNN
+F 1 "MSP432P401R" H 7150 1236 50  0000 C CNN
+F 2 "" H 7150 4450 50  0001 C CNN
+F 3 "" H 7150 4450 50  0001 C CNN
+	1    7150 3250
+	1    0    0    -1
+$EndComp
+Wire Wire Line
+	6550 3000 6300 3000
+Wire Wire Line
+	6300 3000 6300 3300
+Wire Wire Line
+	6300 3300 6150 3300
+Connection ~ 6150 3300
+Wire Wire Line
+	6550 2500 6300 2500
+Wire Wire Line
+	6300 2500 6300 2800
+Wire Wire Line
+	6300 2800 5500 2800
+Wire Wire Line
+	5500 2800 5500 3000
+Connection ~ 5500 2800
+Wire Wire Line
+	4900 2800 4000 2800
+Wire Wire Line
+	4000 2800 4000 3100
+Connection ~ 4900 2800
+Wire Wire Line
+	4900 2800 5500 2800
+Text Label 5500 2900 0    50   ~ 0
++3.3V
+Text Label 4650 2800 0    50   ~ 0
++3.3V
+Text Label 6300 3000 0    50   ~ 0
+ADC_In
+Text Label 5900 3300 0    50   ~ 0
+V_Out
+Text Label 4000 3100 0    50   ~ 0
++3.3V
+Text Label 5100 3200 0    50   ~ 0
+1.65V
+Wire Wire Line
+	4900 3200 5300 3200
+Wire Wire Line
+	5050 2550 5050 3400
+Text Label 5150 3400 0    50   ~ 0
+V_In
 $EndSCHEMATC

Commit message: Updated code and schematic
Parts:
- added C? (x4): 1uF, symbol Device:C
- added D?: 1N4148, Diode_THT:D_DO-35_SOD27_P7.62mm_Horizontal, symbol Diode:1N4148
- added R? (x4): 47kΩ, symbol Device:R_US
- added RTC: DS1337, Package_DIP:DIP-8_W7.62mm, symbol Timer_RTC:DS1337
- added SW?: SW_Push, symbol Switch:SW_Push
- added SW_IN: Signal_In, symbol power:Signal_In
- added Y?: Crystal, symbol Device:Crystal
- MCU: symbol MSP432:MSP432P401R -> Final_Project_Schematic-rescue:MSP432P401R-MSP432
Connections:
- wire segments 26 -> 25
Other:
- moved on the sheet: C, MK, Op-Amp, R

Commit message: complete schematic for project
Parts:
- added J1: LCD connector, symbol Connector:Conn_01x08_Female
- added SCK_LCD: Signal_In, symbol Final_Project_Schematic-rescue:Signal_In-power
- added Vbatt: 3V coin cell, symbol Device:Battery_Cell
- C1, C2: renamed from C?; value 1uF -> 33pF
- C3, C4: renamed from C?; value 1uF -> 0.1uF
- R1, R2: renamed from R?; value 47kΩ -> 4.7kΩ
- R3, R4: renamed from R?; value 47kΩ -> 10kΩ
- RTC: symbol Timer_RTC:DS1337 -> Final_Project_Schematic-rescue:DS1337-Timer_RTC
- SW_IN: symbol power:Signal_In -> Final_Project_Schematic-rescue:Signal_In-power
- gave numbers to parts that had none: 3
Connections:
- net labels added: SCK_LCD, SW_IN, VCC
- wire segments 25 -> 106
Other:
- note added: "CS"
- note added: "DC"
- note added: "GND"
- note added: "LED\n"
- note added: "MOSI"
- note added: "Reset\n"
- note added: "SCK"
- note added: "Vcc"
- moved on the sheet: 32.768KHz, C, C1, C2, C3, C4, D1, MCU, MK, Op-Amp, R, R1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
